File: kicad/rombender.kicad_pcb (KiCad board)
At the start: 2 copper layers, 61.6 x 37.8 mm, 19 parts, among them J3 AVR-ISP-6, J6 Micro_SD_Card, U1 ATmega64A-AU, U2 AP2112K-3.3, U3 TXS0108EPW, U4 28C256, U8 DEVICE, Y1 16MHz

Commit message: a
Connections:
- net /UART_Rx renamed Net-(U1-Pad27)
- net /UART_Tx renamed Net-(U1-Pad28)
- U2 pad 4: GND -> Net-(U2-Pad4)
