File: kicad/rombender.sch (KiCad schematic (older format))
At the start: 19 parts, among them J3 AVR-ISP-6, J6 Micro_SD_Card, U1 ATmega64A-AU, U2 AP2112K-3.3, U3 TXS0108EPW, U4 28C256, U8 DEVICE, Y1 16MHz

Commit message: a
Connections:
- net UART_Rx: no longer names the net of U1.27 (PD2)
- net UART_Tx: no longer names the net of U1.28 (PD3)
- no-connect marks 11 -> 12
Other:
- note added: "JTAG - PF[4:7]"
Changed lines of the file:
@@
 SD Interface
-Wire Wire Line
-	10600 3100 10400 3100
 Wire Wire Line
 	10600 3000 10600 3100
@@
 	1    0    0    -1
 $EndComp
-Wire Wire Line
-	10400 2800 10400 3100
-Connection ~ 10400 3100
-Wire Wire Line
-	10400 3100 10100 3100
 $Comp
 L Device:Crystal_GND24 Y1
@@
 Text Label 3000 2450 0    50   ~ 0
 MISO
-Text Label 3000 4250 0    50   ~ 0
-UART_Tx
-Text Label 3000 4150 0    50   ~ 0
-UART_Rx
 Text Label 1800 3950 2    50   ~ 0
 PDI
@@
 Wire Wire Line
 	9150 750  9150 850
+Wire Wire Line
+	10100 3100 10600 3100
+Text Notes 2150 3700 1    50   ~ 0
+JTAG - PF[4:7]
+NoConn ~ 1800 2050
 $EndSCHEMATC
